File: rgb2hdmi-composite-adapter.brd (EAGLE design)
At the start: 58.4 x 55.9 mm, 24 parts

Commit message: update design
Parts:
- removed U$1: LM319DIP, phantomix-lm319:LM319
- added RESX: 0r, rcl:0207/10
- added U$2: LM319, LM319:DIL14-1
- added VCC@1: TPPAD1-17Y, testpad:P1-17Y
- R1, R2: device pot:CA6V -> pot:B64Y
- moved RES9 11.4 mm to (8.89, 8.89), turned to 90 degrees
- moved RES19 10.5 mm to (21.6, 8.89), turned to 270 degrees
- moved RES17 10.2 mm to (41.9, 8.89), turned to 270 degrees
- moved CAP1 7.62 mm to (16.5, 33.0)
- moved RES18 7.18 mm to (36.8, 8.89), turned to 90 degrees
- moved RES8 5.24 mm to (14.0, 8.89), turned to 270 degrees
- moved CAP7 4.02 mm to (16.5, 25.4), turned to 270 degrees
- moved CAP8 4.02 mm to (34.3, 25.4), turned to 270 degrees
- moved R1 1.27 mm to (11.4, 19.1), turned to 180 degrees
- moved R2 1.27 mm to (39.4, 19.1), turned to 180 degrees
Connections:
- new net VCC@2: RESX.1
- net GND: now also U$2.P2, U$2.P3, U$2.P6, U$2.P8; no longer U$1.3, U$1.6, U$1.8
- net RGB: now also U$2.P12; no longer U$1.12
- net RGBTRIM: now also U$2.P5; no longer U$1.5
- net SYNC: now also U$2.P7; no longer U$1.7
- net SYNCTRIM: now also U$2.P10; no longer U$1.10
- net VCC: now also RESX.2, U$2.P11, U$2.P13, VCC@1.TP; no longer U$1.11
- net VIDEO: now also U$2.P4, U$2.P9; no longer U$1.4, U$1.9
Routing:
- net VCC: track 114.2 -> 151.1 mm
- net SYNC: track 69.7 -> 58.8 mm
- net N$6: track 13.8 -> 5.08 mm
- net VIDEO: track 30.5 -> 38.2 mm
- net N$4: track 11.2 -> 5.08 mm
- net VIDEOIN: track 15.0 -> 8.89 mm
- net RGBTRIM: track 12.5 -> 15.7 mm
- net N$3: track 8.15 -> 5.08 mm
- net SYNCTRIM: track 12.5 -> 15.5 mm
- net N$5: track 3.81 -> 5.08 mm

Commit message: latest, w/new 319
Parts:
- removed U$2: LM319, LM319:DIL14-1
- added U$1: LM319PROPER-DIL-14, LM319:DIL14
- renumbered GND1 to GND@1
Connections:
- net GND: now also U$1.3, U$1.6, U$1.8; no longer U$2.P2, U$2.P3, U$2.P6, U$2.P8
- net RGB: now also U$1.12; no longer U$2.P12
- net RGBTRIM: now also U$1.5; no longer U$2.P5
- net SYNC: now also U$1.7; no longer U$2.P7
- net SYNCTRIM: now also U$1.10; no longer U$2.P10
- net VCC: now also U$1.11; no longer U$2.P11, U$2.P13
- net VIDEO: now also U$1.4, U$1.9; no longer U$2.P4, U$2.P9
Routing:
- net VCC@2: track 0.00 -> 3.96 mm
- net VCC: track 151.1 -> 147.9 mm
- net VIDEO: track 38.2 -> 37.4 mm

Commit message: update for wiki
Parts:
- renumbered RESX to JUMPER
Changed lines of the file:
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@@
 <layer number="17" name="Pads" color="2" fill="1" visible="yes" active="yes"/>
 <layer number="18" name="Vias" color="2" fill="1" visible="yes" active="yes"/>
-<layer number="19" name="Unrouted" color="6" fill="1" visible="yes" active="yes"/>
+<layer number="19" name="Unrouted" color="6" fill="1" visible="no" active="yes"/>
 <layer number="20" name="Dimension" color="24" fill="1" visible="yes" active="yes"/>
-<layer number="21" name="tPlace" color="7" fill="1" visible="no" active="yes"/>
-<layer number="22" name="bPlace" color="7" fill="1" visible="yes" active="yes"/>
+<layer number="21" name="tPlace" color="7" fill="1" visible="yes" active="yes"/>
+<layer number="22" name="bPlace" color="7" fill="1" visible="no" active="yes"/>
 <layer number="23" name="tOrigins" color="15" fill="1" visible="no" active="yes"/>
-<layer number="24" name="bOrigins" color="15" fill="1" visible="yes" active="yes"/>
-<layer number="25" name="tNames" color="7" fill="1" visible="no" active="yes"/>
-<layer number="26" name="bNames" color="7" fill="1" visible="yes" active="yes"/>
+<layer number="24" name="bOrigins" color="15" fill="1" visible="no" active="yes"/>
+<layer number="25" name="tNames" color="7" fill="1" visible="yes" active="yes"/>
+<layer number="26" name="bNames" color="7" fill="1" visible="no" active="yes"/>
 <layer number="27" name="tValues" color="7" fill="1" visible="no" active="yes"/>
 <layer number="28" name="bValues" color="7" fill="1" visible="no" active="yes"/>
@@
 </element>
 <element name="VIDEOIN" library="testpad" library_urn="urn:adsk.eagle:library:385" package="P1-17Y" package3d_urn="urn:adsk.eagle:package:27953/1" value="TPPAD1-17Y" x="7.62" y="31.75" smashed="yes" rot="R90">
-<attribute name="NAME" x="5.08" y="33.02" size="1.27" layer="25" ratio="10" rot="R180" align="top-right"/>
+<attribute name="NAME" x="5.08" y="33.3375" size="1.27" layer="25" ratio="10" rot="R180" align="top-right"/>
 <attribute name="TP_SIGNAL_NAME" value="" x="11.43" y="30.48" size="1" layer="37" rot="R90"/>
 <attribute name="VALUE" x="7.62" y="31.75" size="0.0254" layer="27" rot="R90"/>
 </element>
 <element name="SYNC" library="testpad" library_urn="urn:adsk.eagle:library:385" package="P1-17Y" package3d_urn="urn:adsk.eagle:package:27953/1" value="TPPAD1-17Y" x="53.34" y="26.67" smashed="yes" rot="R90">
-<attribute name="NAME" x="50.8" y="27.94" size="1.27" layer="25" ratio="10"/>
+<attribute name="NAME" x="50.8" y="28.2575" size="1.27" layer="25" ratio="10"/>
 <attribute name="TP_SIGNAL_NAME" value="" x="57.15" y="25.4" size="1" layer="37" rot="R90"/>
 <attribute name="VALUE" x="53.34" y="26.67" size="0.0254" layer="27" rot="R90"/>
 </element>
 <element name="RGB" library="testpad" library_urn="urn:adsk.eagle:library:385" package="P1-17Y" package3d_urn="urn:adsk.eagle:package:27953/1" value="TPPAD1-17Y" x="53.34" y="31.75" smashed="yes" rot="R270">
-<attribute name="NAME" x="50.8" y="33.02" size="1.27" layer="25" ratio="10"/>
+<attribute name="NAME" x="50.8" y="33.3375" size="1.27" layer="25" ratio="10"/>
 <attribute name="TP_SIGNAL_NAME" value="" x="49.53" y="33.02" size="1" layer="37" rot="R270"/>
 <attribute name="VALUE" x="53.34" y="31.75" size="0.0254" layer="27" rot="R270"/>
 </element>
 <element name="VCC" library="testpad" library_urn="urn:adsk.eagle:library:385" package="P1-17Y" package3d_urn="urn:adsk.eagle:package:27953/1" value="TPPAD1-17Y" x="53.34" y="41.91" smashed="yes" rot="R270">
-<attribute name="NAME" x="50.8" y="43.18" size="1.27" layer="25" ratio="10"/>
+<attribute name="NAME" x="50.8" y="43.4975" size="1.27" layer="25" ratio="10"/>
 <attribute name="TP_SIGNAL_NAME" value="" x="49.53" y="43.18" size="1" layer="37" rot="R270"/>
 <attribute name="VALUE" x="53.34" y="41.91" size="0.0254" layer="27" rot="R270"/>
 </element>
 <element name="GND" library="testpad" library_urn="urn:adsk.eagle:library:385" package="P1-17Y" package3d_urn="urn:adsk.eagle:package:27953/1" value="TPPAD1-17Y" x="7.62" y="36.83" smashed="yes" rot="R90">
-<attribute name="NAME" x="5.08" y="38.1" size="1.27" layer="25" ratio="10"/>
+<attribute name="NAME" x="5.08" y="38.4175" size="1.27" layer="25" ratio="10"/>
 <attribute name="TP_SIGNAL_NAME" value="" x="11.43" y="35.56" size="1" layer="37" rot="R90"/>
 <attribute name="VALUE" x="7.62" y="36.83" size="0.0254" layer="27" rot="R90"/>
 </element>
 <element name="GND@1" library="testpad" library_urn="urn:adsk.eagle:library:385" package="P1-17Y" package3d_urn="urn:adsk.eagle:package:27953/1" value="TPPAD1-17Y" x="53.34" y="36.83" smashed="yes" rot="R90">
-<attribute name="NAME" x="50.8" y="38.1" size="1.27" layer="25" ratio="10"/>
+<attribute name="NAME" x="50.8" y="38.4175" size="1.27" layer="25" ratio="10"/>
 <attribute name="TP_SIGNAL_NAME" value="" x="57.15" y="35.56" size="1" layer="37" rot="R90"/>
 <attribute name="VALUE" x="53.34" y="36.83" size="0.0254" layer="27" rot="R90"/>
@@
 <attribute name="VALUE" x="43.18" y="24.511" size="1.27" layer="27" ratio="10" rot="R180"/>
 </element>
-<element name="RESX" library="rcl" library_urn="urn:adsk.eagle:library:334" package="0207/10" package3d_urn="urn:adsk.eagle:package:23491/2" value="0r" x="30.48" y="8.89" smashed="yes" rot="R270">
+<element name="JUMPER" library="rcl" library_urn="urn:adsk.eagle:library:334" package="0207/10" package3d_urn="urn:adsk.eagle:package:23491/2" value="0r" x="30.48" y="8.89" smashed="yes" rot="R270">
 <attribute name="NAME" x="28.956" y="5.842" size="1.27" layer="25" ratio="10" rot="R90"/>
 <attribute name="SPICEPREFIX" value="R" x="30.48" y="8.89" size="1.778" layer="27" rot="R270" display="off"/>
@@
 </element>
 <element name="VCC@1" library="testpad" library_urn="urn:adsk.eagle:library:385" package="P1-17Y" package3d_urn="urn:adsk.eagle:package:27953/1" value="TPPAD1-17Y" x="7.62" y="41.91" smashed="yes" rot="R90">
-<attribute name="NAME" x="5.08" y="43.18" size="1.27" layer="25" ratio="10"/>
+<attribute name="NAME" x="5.08" y="43.4975" size="1.27" layer="25" ratio="10"/>
 <attribute name="TP_SIGNAL_NAME" value="" x="7.62" y="41.91" size="1.778" layer="27" rot="R90" display="off"/>
 <attribute name="VALUE" x="7.62" y="41.91" size="0.0254" layer="27" rot="R90"/>
@@
 <wire x1="45.72" y1="12.065" x2="44.45" y2="10.795" width="0.8128" layer="16"/>
 <wire x1="44.45" y1="10.795" x2="32.385" y2="10.795" width="0.8128" layer="16"/>
-<contactref element="RESX" pad="2"/>
+<contactref element="JUMPER" pad="2"/>
 <contactref element="VCC@1" pad="TP"/>
 <wire x1="21.59" y1="45.72" x2="10.16" y2="45.72" width="0.8128" layer="16"/>
@@
 </signal>
 <signal name="VCC@2">
-<contactref element="RESX" pad="1"/>
+<contactref element="JUMPER" pad="1"/>
 <wire x1="30.48" y1="13.97" x2="30.48" y2="12.7" width="0.8128" layer="16"/>
 <wire x1="30.48" y1="12.7" x2="32.385" y2="10.795" width="0.8128" layer="16"/>
